File: hardware/alaya-vijnana/alaya-vijnana.kicad_pcb (KiCad board)
At the start: 4 copper layers, 180 parts, among them J1 Bat, J2 USB_C_Receptacle_USB2.0_16P, J3 Bat, J4 USB_C_Receptacle_USB2.0_16P, J5 MAIN_CONN, J6 MAIN_CONN, J7 CLUSTER_CONN, J8 CLUSTER_CONN, SW1 Power_Switch, SW10 MX HotSwap, SW11 MX HotSwap, SW12 MX HotSwap, SW13 MX HotSwap, SW14 MX HotSwap, SW15 MX HotSwap, SW16 MX HotSwap, SW17 MX HotSwap, SW18 MX HotSwap, SW19 MX HotSwap, SW2 MX HotSwap, SW20 MX HotSwap, SW21 MX HotSwap, SW22 MX HotSwap, SW23 Power_Switch, SW24 MX HotSwap, SW25 MX HotSwap, SW26 MX HotSwap, SW27 MX HotSwap, SW28 MX HotSwap, SW29 MX HotSwap, SW3 MX HotSwap, SW30 MX HotSwap, SW31 MX HotSwap, SW32 MX HotSwap, SW33 MX HotSwap, SW34 MX HotSwap, SW35 MX HotSwap, SW36 MX HotSwap, SW37 MX HotSwap, SW38 MX HotSwap, SW39 MX HotSwap, SW4 MX HotSwap, SW40 MX HotSwap, SW41 MX HotSwap, SW42 MX HotSwap, SW43 MX HotSwap, SW44 MX HotSwap, SW5 MX HotSwap, SW6 MX HotSwap, SW7 MX HotSwap, SW8 MX HotSwap, SW9 MX HotSwap, U1 nRF52840, U2 BQ24075RGT, U3 XC6220B331MR, U4 nRF52840, U5 XC6220B331MR, U6 BQ24075RGT, X1 32.768kHz, X2 32.768kHz, Y1 32Mhz, Y2 32Mhz

Commit message: left side wired up
Parts:
- C1, C11, C12, C2, C23, C24, C25, C3, C4, C5, C6, C7, C8, C9, L2, L3, L4, R1, R2, R3, R5, TP1, U1, U2, U3, X1, Y1: moved to B.Cu
- L1: footprint Inductor_SMD:L_0603_1608Metric_Pad1.05x0.95mm_HandSolder -> Inductor_SMD:L_0402_1005Metric_Pad0.77x0.64mm_HandSolder; moved to B.Cu
- moved R2 114.9 mm to (102.8, 99.8), turned to 180 degrees
- moved TP1 114.1 mm to (100.2, 96.5), turned to 180 degrees
- moved R1 113.5 mm to (98.5, 93.3), turned to 180 degrees
- moved L4 66.3 mm to (123.6, 103.4)
- moved L2 63.2 mm to (128.9, 103.3), turned to 90 degrees
- moved L3 60.8 mm to (130.4, 103.3), turned to -90 degrees
- moved C3 45.7 mm to (111.0, 99.0), turned to 90 degrees
- moved C5 42.8 mm to (113.2, 101.5)
- moved C4 41.0 mm to (114.0, 95.5)
- moved C23 28.5 mm to (134.5, 103.2)
- moved C1 28.5 mm to (128.3, 90.2), turned to 90 degrees
- moved C8 28.2 mm to (124.6, 86.6), turned to 180 degrees
- moved C6 27.1 mm to (126.9, 92.9), turned to 0 degrees
- moved L1 26.4 mm to (126.0, 91.0), turned to 90 degrees
- moved C7 26.4 mm to (124.6, 88.4), turned to 180 degrees
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Connections:
- C5 pad 1: unconnected-(C5-Pad1) -> L_BAT-
- J3 pad 2: BAT- -> L_BAT-
- U1 pad A8: unconnected-(U1-AIN7/P0.31-PadA8) -> L_COL5
- U1 pad B9: unconnected-(U1-AIN6/P0.30-PadB9) -> L_COL6
- U1 pad G1: unconnected-(U1-P0.26-PadG1) -> L_COL0
- U1 pad J1: unconnected-(U1-AIN2/P0.04-PadJ1) -> L_COL1
- U1 pad L1: unconnected-(U1-P0.06-PadL1) -> L_COL2
- U1 pad N1: unconnected-(U1-P0.08-PadN1) -> L_COL3
- U1 pad P2: unconnected-(U1-P1.08-PadP2) -> L_COL4
- U1 pad R1: unconnected-(U1-TRACEDATA3/P1.09-PadR1) -> L_ROW2
- U1 pad T2: unconnected-(U1-TRACEDATA2/P0.11-PadT2) -> L_ROW0
- U1 pad U1: unconnected-(U1-TRACEDATA1/P0.12-PadU1) -> L_ROW1
- U2 pad 6: VDDH -> L_VDDH
- Y1 pad 4: L_BAT- -> (no net)
Routing:
- net L_COL0: track 38.1 -> 140.9 mm, vias 3 -> 4
- net L_ROW0: track 92.1 -> 177.5 mm, vias 0 -> 4
- net L_COL1: track 38.1 -> 117.8 mm, vias 3 -> 4
- net L_VBUS: track 0.00 -> 71.9 mm, vias 0 -> 3
- net L_VDDH: track 0.00 -> 71.3 mm, vias 0 -> 1
- net L_ROW1: track 95.2 -> 164.7 mm, vias 0 -> 4
- net L_COL2: track 38.1 -> 101.6 mm, vias 3 -> 4
- net L_COL4: track 0.00 -> 54.2 mm, vias 3 -> 4
- net Net-(LED1-K): track 0.00 -> 43.6 mm, vias 0 -> 1
- net L_VBAT: track 0.00 -> 39.4 mm, vias 0 -> 1
- net L_COL3: track 38.1 -> 76.0 mm, vias 3 -> 4
- net L_ROW2: track 96.1 -> 130.4 mm, vias 0 -> 2
- net L_D-: track 0.00 -> 34.3 mm, vias 0 -> 5
- net L_D+: track 0.00 -> 32.8 mm, vias 0 -> 4
- net L_COL5: track 0.00 -> 32.7 mm, vias 0 -> 1
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Other:
- board outline added: 354 x 168.2 mm

Commit message: finished
Parts:
- C26, C27, C28, C29, C30, C31, C32, C33, C34, C35, C36, C37, C38, C39, C40, C41, C42, C43, C44, C45, C46, C47, C48, C49, C50, J3, J4, J6, L5, L6, L7, L8, R10, R11, R13, R8, R9, TP2, U4, U5, U6, X2, Y2: moved to B.Cu
- moved L8 350.8 mm to (215.9, 101.7), turned to 180 degrees
- moved Y2 341.4 mm to (221.7, 91.6)
- moved L5 340.4 mm to (226.8, 95.4), turned to 90 degrees
- moved L7 338.6 mm to (229.0, 105.4)
- moved L6 338.6 mm to (228.4, 95.4), turned to -90 degrees
- moved X2 333.1 mm to (228.8, 101.4), turned to 90 degrees
- moved J4 331.6 mm to (219.4, 84.6), turned to 90 degrees
- moved R14 329.5 mm to (216.5, 79.7), turned to 90 degrees
- moved LED2 328.3 mm to (215.7, 74.7)
- moved C49 327.5 mm to (214.9, 99.7), turned to 180 degrees
- moved R12 327.3 mm to (218.7, 74.7), turned to -90 degrees
- moved C50 325.5 mm to (216.6, 97.3), turned to 90 degrees
- moved R13 324.9 mm to (221.2, 83.5), turned to -90 degrees
- moved C48 324.9 mm to (217.8, 100.7), turned to 90 degrees
- moved C35 322.7 mm to (216.8, 103.2)
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Connections:
- C46 pad 1: unconnected-(C46-Pad1) -> L_BAT-
- U4 pad AC21: unconnected-(U4-P0.25-PadAC21) -> COL4
- U4 pad AD12: unconnected-(U4-P0.17-PadAD12) -> ROW0
- U4 pad AD16: unconnected-(U4-P0.20-PadAD16) -> ROW1
- U4 pad AD18: unconnected-(U4-P0.22-PadAD18) -> ROW2
- U4 pad AD20: unconnected-(U4-P0.24-PadAD20) -> COL6
- U4 pad AD22: unconnected-(U4-TRACEDATA0/P1.00-PadAD22) -> COL5
- U4 pad R24: unconnected-(U4-P1.06-PadR24) -> COL0
- U4 pad U24: unconnected-(U4-P1.04-PadU24) -> COL1
- U4 pad W24: unconnected-(U4-P1.02-PadW24) -> COL2
- U4 pad Y23: unconnected-(U4-P1.01-PadY23) -> COL3
Routing:
- net ROW1: track 0.00 -> 196.0 mm, vias 0 -> 4
- net ROW0: track 0.00 -> 188.1 mm, vias 0 -> 3
- net COL0: track 0.00 -> 172.0 mm, vias 0 -> 4
- net COL1: track 0.00 -> 151.5 mm, vias 0 -> 4
- net COL2: track 0.00 -> 129.6 mm, vias 0 -> 4
- net ROW2: track 0.00 -> 124.0 mm, vias 0 -> 2
- net COL3: track 0.00 -> 101.3 mm, vias 0 -> 4
- net COL4: track 0.00 -> 79.2 mm, vias 0 -> 4
- net VDDH: track 0.00 -> 61.8 mm, vias 0 -> 1
- net VBUS: track 0.00 -> 56.2 mm, vias 0 -> 1
- net RF: track 0.00 -> 34.2 mm
- net Net-(U6-ISET): track 0.00 -> 32.2 mm, vias 0 -> 2
- net D-: track 0.00 -> 30.2 mm, vias 0 -> 1
- net COL5: track 0.00 -> 30.0 mm, vias 0 -> 2
- net D+: track 0.00 -> 29.4 mm, vias 0 -> 1
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- added copper zone on In1.Cu, net L_BAT-
Other:
- board size 354 x 168.2 mm -> 235.7 x 146.6 mm

Commit message: fixed everything
Connections:
- Y1 pad 4: (no net) -> L_BAT-
Routing:
- net L_COL4: track 55.4 -> 54.4 mm
- net D-: track 30.2 -> 29.6 mm
- net D+: track 29.4 -> 28.9 mm
- net L_BAT-: vias 74 -> 76
- net VDD_NRF: vias 3 -> 2

Commit message: split into parts
Parts:
- moved R12 0.80 mm to (219.5, 74.7)
- moved LED2 0.59 mm to (216.0, 74.2)
- moved SW23 0.22 mm to (220.7, 69.5)
Routing:
- net VDDH: track 61.6 -> 60.8 mm
Other:
- board text added: "JLCJLCJLC"

Commit message: production stuff
Parts:
- added SW45: SW_Push, Button_Switch_SMD:SW_Push_1P1T_NO_CK_KMR2, F.Cu at (185.8, 61.4)
- added SW46: SW_Push, Button_Switch_SMD:SW_Push_1P1T_NO_CK_KMR2, F.Cu at (226.3, 61.2)
- moved D17 19.4 mm to (165.7, 165.4), turned to 0 degrees
- moved D18 19.3 mm to (146.9, 165.5), turned to 0 degrees
- turned SW18 to -90 degrees
- turned SW19 to -90 degrees
Connections:
- U1 pad AC13: unconnected-(U1-P0.18/~{RESET}-PadAC13) -> Net-(U1-P0.18/~{RESET})
- U4 pad AC13: unconnected-(U4-P0.18/~{RESET}-PadAC13) -> Net-(U4-P0.18/~{RESET})
- Y1 pad 4: L_BAT- -> (no net)
Routing:
- net Net-(U1-P0.18/~{RESET}): track 0.00 -> 48.3 mm, vias 0 -> 3
- net Net-(U4-P0.18/~{RESET}): track 0.00 -> 47.1 mm, vias 0 -> 3
- net LC_COL5: track 60.7 -> 95.6 mm
- net LC_COL6: track 83.8 -> 64.7 mm, vias 3 -> 2
- net LC_ROW2: track 67.6 -> 81.2 mm
- net L_BAT-: track 64.5 -> 72.7 mm, vias 76 -> 80
- net LC_ROW1: track 57.1 -> 52.1 mm
- net L_BAT+: track 30.6 -> 28.5 mm
- net L_D+: track 35.6 -> 34.0 mm, vias 4 -> 2
- net L_D-: track 36.9 -> 35.4 mm, vias 5 -> 2
