File: hardware/alaya-vijnana/left-cluster.kicad_pcb (KiCad board)
At the start: 4 copper layers, 57.4 x 57.4 mm, 13 parts, among them J8 CLUSTER_CONN, SW17 MX HotSwap, SW18 MX HotSwap, SW19 MX HotSwap, SW20 MX HotSwap, SW21 MX HotSwap, SW22 MX HotSwap

Commit message: production stuff
Parts:
- moved D16 70.5 mm to (233.3, 151.6)
- moved D19 70.5 mm to (252.4, 151.8)
- moved D21 70.5 mm to (252.4, 189.9)
- moved J8 70.5 mm to (226.7, 142.5)
- moved SW17 70.5 mm to (241.6, 146.5)
- moved SW18 70.5 mm to (241.6, 175.1), turned to -90 degrees
- moved SW19 70.5 mm to (222.5, 175.1), turned to -90 degrees
- moved SW20 70.5 mm to (260.6, 146.5)
- moved SW21 70.5 mm to (260.6, 165.5)
- moved SW22 70.5 mm to (260.6, 184.6)
- moved D20 70.5 mm to (252.5, 170.8)
- moved D18 62.0 mm to (217.4, 167.0), turned to 0 degrees
- moved D17 61.8 mm to (236.2, 166.9), turned to 0 degrees
Routing:
- net LC_COL5: track 60.7 -> 95.6 mm
- net LC_COL6: track 83.8 -> 64.7 mm, vias 3 -> 2
- net LC_ROW2: track 67.6 -> 81.2 mm
- net LC_ROW1: track 57.1 -> 52.1 mm
