File: hardware/alaya-vijnana/right-main.kicad_pcb (KiCad board)
At the start: 4 copper layers, 113.1 x 86.7 mm, 77 parts, among them J3 Bat, J4 USB_C_Receptacle_USB2.0_16P, J6 MAIN_CONN, SW23 Power_Switch, SW24 MX HotSwap, SW25 MX HotSwap, SW26 MX HotSwap, SW27 MX HotSwap, SW28 MX HotSwap, SW29 MX HotSwap, SW30 MX HotSwap, SW31 MX HotSwap, SW32 MX HotSwap, SW33 MX HotSwap, SW34 MX HotSwap, SW35 MX HotSwap, SW36 MX HotSwap, SW37 MX HotSwap, SW38 MX HotSwap, U4 nRF52840, U5 XC6220B331MR, U6 BQ24075RGT, X2 32.768kHz, Y2 32Mhz

Commit message: added firmware
Routing:
- added copper zone on In2.Cu, net L_BAT-
Other:
- board text added: "JLCJLCJLCJLC"
- board text removed: "JLCJLCJLC"
Changed lines of the file:
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@@
 		(layer "Edge.Cuts")
 	)
-	(gr_text "JLCJLCJLC"
+	(gr_text "JLCJLCJLCJLC"
 		(at 241.9 127.2 0)
 		(layer "B.SilkS")
@@
 		(net 105)
 		(net_name "L_BAT-")
-		(layer "In1.Cu")
+		(layers "In1.Cu" "In2.Cu")
 		(hatch edge 0.5)
 		(connect_pads

Commit message: production stuff
Parts:
- removed SW23: Power_Switch, Button_Switch_THT:SW_E-Switch_EG1224_SPDT_Angled
- added SW46: SW_Push, Button_Switch_SMD:SW_Push_1P1T_NO_CK_KMR2, F.Cu at (216.0, 89.0)
- moved D24 29.6 mm to (295.7, 141.9)
- moved D27 29.6 mm to (276.7, 132.4)
- moved D33 29.6 mm to (238.7, 137.1)
- moved D36 29.6 mm to (219.5, 141.9)
- moved R8 29.6 mm to (234.1, 131.2)
- moved C26 29.6 mm to (216.5, 135.8)
- moved C27 29.6 mm to (215.0, 135.8)
- moved C30 29.6 mm to (219.1, 134.9)
- moved C32 29.6 mm to (215.9, 120.3)
- moved C33 29.6 mm to (219.1, 126.9)
- moved C36 29.6 mm to (213.5, 135.8)
- moved C37 29.6 mm to (219.0, 131.5)
- moved C38 29.6 mm to (219.1, 136.3)
- moved C39 29.6 mm to (213.5, 123.4)
- moved C40 29.6 mm to (215.0, 123.4)
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Connections:
- U4 pad AC13: unconnected-(U4-P0.18/~{RESET}-PadAC13) -> Net-(U4-P0.18/~{RESET})
Routing:
- net Net-(U4-P0.18/~{RESET}): track 0.00 -> 47.1 mm, vias 0 -> 3
- net L_BAT-: track 22.0 -> 26.1 mm, vias 35 -> 37
- removed copper zone on In2.Cu, net L_BAT-
Other:
- outline, holes or cut-outs redrawn
- board text added: "JLCJLCJLC"
- board text added: "SW23"
- board text removed: "JLCJLCJLCJLC"
