File: hardware/_restore_backup_2026-06-10T13-15-52-418/alaya-vijnana.kicad_pcb (KiCad board)
At the start: 2 copper layers, 77 parts, among them J1 Debug/Flash, J3 Bat, J4 USB_C_Receptacle_USB2.0_16P, J6 MAIN_CONN, J7 CLUSTER_CONN, SW1 MX HotSwap, SW10 MX HotSwap, SW11 MX HotSwap, SW12 MX HotSwap, SW13 MX HotSwap, SW14 MX HotSwap, SW15 MX HotSwap, SW16 MX HotSwap, SW17 MX HotSwap, SW18 MX HotSwap, SW19 MX HotSwap, SW2 MX HotSwap, SW20 MX HotSwap, SW21 MX HotSwap, SW3 MX HotSwap, SW4 MX HotSwap, SW5 MX HotSwap, SW6 MX HotSwap, SW7 MX HotSwap, SW8 MX HotSwap, SW9 MX HotSwap, U1 nRF52840_E73-2G4M08S1C, U6 BQ24075RGT, X2 32.768kHz

Commit message: lots more routing
Parts:
- C2, C26, C27, C28, C29, C30, R14: moved to F.Cu
- moved TP2 140.9 mm to (262.7, 105.0)
- moved R9 135.5 mm to (254.8, 109.6)
- moved L7 132.7 mm to (255.6, 61.9), turned to 0 degrees
- moved R8 130.4 mm to (254.8, 104.8)
- moved X2 119.5 mm to (244.8, 85.4), turned to 0 degrees
- moved R14 118.7 mm to (235.2, 81.3), turned to 0 degrees
- moved R13 113.4 mm to (235.2, 78.8), turned to 0 degrees
- moved F1 111.9 mm to (230.9, 78.8), turned to 0 degrees
- moved C30 106.7 mm to (226.5, 73.8), turned to 0 degrees
- moved C29 106.7 mm to (226.5, 71.3), turned to 0 degrees
- moved C28 106.1 mm to (223.6, 86.5), turned to 0 degrees
- moved C2 102.9 mm to (222.2, 73.8), turned to 0 degrees
- moved C27 102.0 mm to (222.2, 78.8), turned to 0 degrees
- moved C42 101.6 mm to (226.5, 81.3)
- moved C26 100.3 mm to (222.2, 76.3), turned to 0 degrees
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Connections:
- U1 pad 15: unconnected-(U1-P0.05/AIN3-Pad15) -> SLC
- U1 pad 22: unconnected-(U1-P0.07-Pad22) -> SDA
Routing:
- net VBUS: track 39.9 -> 0.00 mm, vias 3 -> 0
- net COL4: track 38.1 -> 0.00 mm
- net D-: track 23.3 -> 0.00 mm
- net D+: track 23.2 -> 0.00 mm
- net VDD_NRF: track 22.8 -> 0.00 mm, vias 1 -> 0
- net VBAT: track 18.6 -> 0.00 mm
- net VDDH: track 16.7 -> 0.00 mm, vias 1 -> 0
- net Net-(LED2-K): track 12.6 -> 0.00 mm
- net Net-(F1-Pad1): track 9.54 -> 0.00 mm
- net Net-(U1-P0.00/XL1): track 7.39 -> 0.00 mm, vias 1 -> 0
- net Net-(U1-P0.01/XL2): track 7.11 -> 0.00 mm, vias 1 -> 0
- net BAT-: track 3.43 -> 0.00 mm, vias 2 -> 0
- net Net-(U1-DCCH): track 3.03 -> 0.00 mm, vias 1 -> 0
- net Net-(J4-CC1): track 2.08 -> 0.00 mm
- net Net-(J4-CC2): track 1.82 -> 0.00 mm
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