File: hardware/_restore_backup_2026-06-10T13-15-52-418/alaya-vijnana.kicad_sch (KiCad schematic)
At the start: 31 parts, among them J1 Debug/Flash, J3 Bat, J4 USB_C_Receptacle_USB2.0_16P, U1 nRF52840_E73-2G4M08S1C, U6 BQ24075RGT, X2 32.768kHz

Commit message: lots more routing
Connections:
- net COL0: now also U1.42 (P1.06); no longer U1.1 (P1.11)
- net COL1: now also U1.17 (P1.09); no longer U1.2 (P1.10)
- net COL2: now also U1.2 (P1.10); no longer U1.3 (P0.03/AIN1)
- net COL3: now also U1.1 (P1.11); no longer U1.42 (P1.06)
- net COL4: now also U1.6 (P1.13); no longer U1.22 (P0.07)
- net COL5: now also U1.33 (P0.13); no longer U1.17 (P1.09)
- net COL6: now also U1.28 (P0.15); no longer U1.10 (P0.30/AIN6)
- net ROW0: now also U1.36 (P1.00)
- net ROW1: now also U1.38 (P1.02)
- net ROW2: now also U1.40 (P1.04)
- net SLC: now reaches U1.15 (P0.05/AIN3)
- new net SDA: U1.22 (P0.07)
- no-connect marks 22 -> 6
Changed lines of the file:
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@@
-	)
-	(no_connect
-		(at 90.17 54.61)
-	)
-	(no_connect
-		(at 90.17 52.07)
 	)
 	(no_connect
@@
 	)
 	(no_connect
-		(at 90.17 80.01)
-	)
-	(no_connect
-		(at 44.45 107.95)
-	)
-	(no_connect
-		(at 44.45 87.63)
-	)
-	(no_connect
-		(at 44.45 100.33)
-	)
-	(no_connect
 		(at 162.56 54.61)
-	)
-	(no_connect
-		(at 44.45 82.55)
-	)
-	(no_connect
-		(at 90.17 59.69)
 	)
 	(no_connect
@@
 	)
 	(no_connect
-		(at 44.45 90.17)
-	)
-	(no_connect
-		(at 44.45 102.87)
-	)
-	(no_connect
-		(at 44.45 97.79)
-	)
-	(no_connect
-		(at 44.45 105.41)
-	)
-	(no_connect
-		(at 90.17 64.77)
-	)
-	(no_connect
 		(at 143.51 105.41)
-	)
-	(no_connect
-		(at 90.17 46.99)
-	)
-	(no_connect
-		(at 90.17 77.47)
 	)
 	(no_connect
 		(at 247.65 54.61)
 	)
-	(no_connect
-		(at 90.17 57.15)
-	)
 	(wire
 		(pts
@@
 	(wire
 		(pts
+			(xy 43.18 85.09) (xy 44.45 85.09)
+		)
+		(stroke
+			(width 0)
+			(type default)
+		)
+	)
+	(wire
+		(pts
 			(xy 193.04 49.53) (xy 194.31 49.53)
 		)
@@
 	(wire
 		(pts
+			(xy 90.17 54.61) (xy 91.44 54.61)
+		)
+		(stroke
+			(width 0)
+			(type default)
+		)
+	)
+	(wire
+		(pts
 			(xy 187.96 44.45) (xy 198.12 44.45)
 		)
@@
 	(global_label "COL4"
 		(shape bidirectional)
-		(at 44.45 85.09 180)
+		(at 90.17 107.95 0)
 		(fields_autoplaced yes)
 		(effects
@@
 				(size 1.27 1.27)
 			)
-			(justify right)
-		)
-		(property "Intersheetrefs" "${INTERSHEET_REFS}"
-			(at 35.5154 85.09 0)
-			(hide yes)
-			(show_name no)
-			(do_not_autoplace no)
-			(effects
-				(font
-					(size 1.27 1.27)
-				)
-				(justify right)
+			(justify left)
+		)
+		(property "Intersheetrefs" "${INTERSHEET_REFS}"
+			(at 99.1046 107.95 0)
+			(hide yes)
+			(show_name no)
+			(do_not_autoplace no)
+			(effects
+				(font
+					(size 1.27 1.27)
+				)
+				(justify left)
 			)
 		)
@@
 	(global_label "COL0"
 		(shape bidirectional)
-		(at 90.17 105.41 0)
+		(at 90.17 97.79 0)
 		(fields_autoplaced yes)
 		(effects
@@
 		)
 		(property "Intersheetrefs" "${INTERSHEET_REFS}"
-			(at 99.1046 105.41 0)
+			(at 99.1046 97.79 0)
 			(hide yes)
 			(show_name no)
@@
 	(global_label "COL5"
 		(shape bidirectional)
-		(at 90.17 100.33 0)
+		(at 44.45 92.71 180)
 		(fields_autoplaced yes)
 		(effects
@@
 				(size 1.27 1.27)
 			)
-			(justify left)
-		)
-		(property "Intersheetrefs" "${INTERSHEET_REFS}"
-			(at 99.1046 100.33 0)
-			(hide yes)
-			(show_name no)
-			(do_not_autoplace no)
-			(effects
-				(font
-					(size 1.27 1.27)
-				)
-				(justify left)
+			(justify right)
+		)
+		(property "Intersheetrefs" "${INTERSHEET_REFS}"
+			(at 35.5154 92.71 0)
+			(hide yes)
+			(show_name no)
+			(do_not_autoplace no)
+			(effects
+				(font
+					(size 1.27 1.27)
+				)
+				(justify right)
 			)
 		)
@@
 	(global_label "COL3"
 		(shape bidirectional)
-		(at 90.17 97.79 0)
+		(at 90.17 105.41 0)
 		(fields_autoplaced yes)
 		(effects
@@
 		)
 		(property "Intersheetrefs" "${INTERSHEET_REFS}"
-			(at 99.1046 97.79 0)
+			(at 99.1046 105.41 0)
 			(hide yes)
 			(show_name no)
@@
 	(global_label "COL6"
 		(shape bidirectional)
-		(at 90.17 62.23 0)
+		(at 44.45 95.25 180)
 		(fields_autoplaced yes)
 		(effects
@@
 				(size 1.27 1.27)
 			)
-			(justify left)
-		)
-		(property "Intersheetrefs" "${INTERSHEET_REFS}"
-			(at 99.1046 62.23 0)
-			(hide yes)
-			(show_name no)
-			(do_not_autoplace no)
-			(effects
-				(font
-					(size 1.27 1.27)
-				)
-				(justify left)
+			(justify right)
+		)
+		(property "Intersheetrefs" "${INTERSHEET_REFS}"
+			(at 35.5154 95.25 0)
+			(hide yes)
+			(show_name no)
+			(do_not_autoplace no)
+			(effects
+				(font
+					(size 1.27 1.27)
+				)
+				(justify right)
 			)
 		)
@@
 	(global_label "COL2"
 		(shape bidirectional)
-		(at 90.17 49.53 0)
+		(at 90.17 102.87 0)
 		(fields_autoplaced yes)
 		(effects
@@
 		)
 		(property "Intersheetrefs" "${INTERSHEET_REFS}"
-			(at 99.1046 49.53 0)
+			(at 99.1046 102.87 0)
+			(hide yes)
+			(show_name no)
+			(do_not_autoplace no)
+			(effects
+				(font
+					(size 1.27 1.27)
+				)
+				(justify left)
+			)
+		)
+	)
+	(global_label "SLC"
+		(shape bidirectional)
+		(at 91.44 54.61 0)
+		(fields_autoplaced yes)
+		(effects
+			(font
+				(size 0.762 0.762)
+			)
+			(justify left)
+		)
+		(property "Intersheetrefs" "${INTERSHEET_REFS}"
+			(at 96.0028 54.61 0)
 			(hide yes)
 			(show_name no)
@@
 	(global_label "COL1"
 		(shape bidirectional)
-		(at 90.17 102.87 0)
+		(at 90.17 100.33 0)
 		(fields_autoplaced yes)
 		(effects
@@
 		)
 		(property "Intersheetrefs" "${INTERSHEET_REFS}"
-			(at 99.1046 102.87 0)
+			(at 99.1046 100.33 0)
 			(hide yes)
 			(show_name no)
@@
 		)
 	)
+	(global_label "SDA"
+		(shape bidirectional)
+		(at 43.18 85.09 180)
+		(fields_autoplaced yes)
+		(effects
+			(font
+				(size 0.762 0.762)
+			)
+			(justify right)
+		)
+		(property "Intersheetrefs" "${INTERSHEET_REFS}"
+			(at 38.581 85.09 0)
+			(hide yes)
+			(show_name no)
+			(do_not_autoplace no)
+			(effects
+				(font
+					(size 1.27 1.27)
+				)
+				(justify right)
+			)
+		)
+	)
 	(global_label "VBUS"
 		(shape bidirectional)
@@
 	(global_label "ROW0"
 		(shape bidirectional)
-		(at 127 118.11 0)
+		(at 90.17 90.17 0)
 		(fields_autoplaced yes)
 		(effects
@@
 		)
 		(property "Intersheetrefs" "${INTERSHEET_REFS}"
-			(at 136.3579 118.11 0)
+			(at 99.5279 90.17 0)
 			(hide yes)
 			(show_name no)
@@
 	(global_label "ROW2"
 		(shape bidirectional)
-		(at 127 123.19 0)
+		(at 90.17 95.25 0)
 		(fields_autoplaced yes)
 		(effects
@@
 		)
 		(property "Intersheetrefs" "${INTERSHEET_REFS}"
-			(at 136.3579 123.19 0)
+			(at 99.5279 95.25 0)
 			(hide yes)
 			(show_name no)
@@
 	(global_label "ROW1"
 		(shape bidirectional)
-		(at 127 120.65 0)
+		(at 90.17 92.71 0)
 		(fields_autoplaced yes)
 		(effects
@@
 		)
 		(property "Intersheetrefs" "${INTERSHEET_REFS}"
-			(at 136.3579 120.65 0)
-			(hide yes)
-			(show_name no)
+			(at 99.5279 92.71 0)
+			(hide yes)
+			(show_name no)
