File: hardware/alaya-vijnana.kicad_pcb (KiCad board)
At the start: 2 copper layers, 77 parts, among them J1 Debug/Flash, J3 Bat, J4 USB_C_Receptacle_USB2.0_16P, J6 MAIN_CONN, J7 CLUSTER_CONN, SW1 MX HotSwap, SW10 MX HotSwap, SW11 MX HotSwap, SW12 MX HotSwap, SW13 MX HotSwap, SW14 MX HotSwap, SW15 MX HotSwap, SW16 MX HotSwap, SW17 MX HotSwap, SW18 MX HotSwap, SW19 MX HotSwap, SW2 MX HotSwap, SW20 MX HotSwap, SW21 MX HotSwap, SW3 MX HotSwap, SW4 MX HotSwap, SW5 MX HotSwap, SW6 MX HotSwap, SW7 MX HotSwap, SW8 MX HotSwap, SW9 MX HotSwap, U1 nRF52840_E73-2G4M08S1C, U6 BQ24075RGT, X2 32.768kHz

Commit message: left side done
Parts:
- J1: moved to F.Cu
- J3, J6, J7, POWER-SW1, R8, R9, TP2: moved to B.Cu
- moved J3 151.1 mm to (116.3, 58.0), turned to 90 degrees
- moved R8 57.9 mm to (122.6, 49.3), turned to 90 degrees
- moved R9 52.9 mm to (122.6, 54.4), turned to 90 degrees
- moved TP2 52.2 mm to (125.9, 51.9), turned to 90 degrees
- moved J1 51.4 mm to (131.8, 90.0), turned to 180 degrees
- moved RESET-SW1 36.6 mm to (138.6, 57.8), turned to 180 degrees
- moved POWER-SW1 7.06 mm to (134.5, 40.5), turned to -90 degrees
- moved J7 5.25 mm to (81.2, 123.2)
- moved J6 5.10 mm to (123.4, 88.5)
- moved LED2 1.29 mm to (138.0, 54.9)
- moved R12 1.29 mm to (137.9, 53.2)
Connections:
- U1 pad 1: COL3 -> COL0
- U1 pad 10: unconnected-(U1-P0.30/AIN6-Pad10) -> COL6
- U1 pad 12: unconnected-(U1-P0.26-Pad12) -> ROW1
- U1 pad 14: unconnected-(U1-P0.06-Pad14) -> ROW2
- U1 pad 15: unconnected-(U1-P0.05/AIN3-Pad15) -> ROW0
- U1 pad 17: COL1 -> unconnected-(U1-P1.09-Pad17)
- U1 pad 2: COL2 -> COL1
- U1 pad 28: COL6 -> unconnected-(U1-P0.15-Pad28)
- U1 pad 3: unconnected-(U1-P0.03/AIN1-Pad3) -> COL2
- U1 pad 33: COL5 -> unconnected-(U1-P0.13-Pad33)
- U1 pad 36: ROW0 -> unconnected-(U1-P1.00-Pad36)
- U1 pad 38: ROW1 -> unconnected-(U1-P1.02-Pad38)
- U1 pad 40: ROW2 -> unconnected-(U1-P1.04-Pad40)
- U1 pad 42: COL0 -> unconnected-(U1-P1.06-Pad42)
- U1 pad 6: COL4 -> COL3
- U1 pad 7: unconnected-(U1-P0.02/AIN0-Pad7) -> COL4
- U1 pad 9: unconnected-(U1-P0.31/AIN7-Pad9) -> COL5
Routing:
- net COL0: track 38.1 -> 166.5 mm, vias 0 -> 1
- net COL1: track 38.1 -> 143.5 mm, vias 0 -> 1
- net COL2: track 38.1 -> 127.0 mm, vias 0 -> 1
- net ROW2: track 93.3 -> 154.5 mm, vias 0 -> 1
- net COL3: track 38.1 -> 97.0 mm, vias 0 -> 1
- net ROW0: track 92.4 -> 146.9 mm, vias 0 -> 1
- net RESET: track 0.00 -> 44.5 mm, vias 0 -> 2
- net ROW1: track 93.1 -> 135.6 mm, vias 0 -> 1
- net BAT+: track 0.00 -> 39.3 mm
- net BAT-: track 3.43 -> 36.1 mm, vias 2 -> 21
- net COL4: track 38.1 -> 70.5 mm, vias 0 -> 1
- net Net-(U6-ISET): track 0.00 -> 29.2 mm, vias 0 -> 3
- net SWDCLK: track 0.00 -> 27.6 mm, vias 0 -> 1
- net VDD_NRF: track 22.8 -> 49.8 mm, vias 1 -> 2
- net SWDIO: track 0.00 -> 24.8 mm, vias 0 -> 1
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- added copper zone on B.Cu, net BAT-
- added copper zone on F.Cu, net BAT-
Other:
- board outline added: 116.8 x 71.7 mm
